File: SOURCES/KICAD/ADAT-IO-x4.sch (KiCad schematic (older format))
At the start: 95 parts, among them IC11 XC6SLX9-TQ144, IC12 AT25F2048N, IC13 LTC3419, IC14 74AHC14, IC20 ADM811TARTZ, SW1 NT04, SW2 5MS1, X1 PLR135/T10, X10 PLT133/T10W, X11 IDC-2x32, X12 IDC-2x8, X13 IDC-2x8, X2 PLR135/T10, X3 PLR135/T10, X4 PLR135/T10, X5 PLT133/T10W, X6 CONN_02X07, X7 BNC, X8 PLT133/T10W, X9 PLT133/T10W

Commit message: PCB layout prototype
Parts:
- removed C114: 100n, rklib:C0805-X7R, symbol C
- removed D10, D9: 1N4148, Diodes_SMD:MiniMELF_Standard, symbol D
- removed IC14: 74AHC14, Housings_SOIC:SOIC-14_3.9x8.7mm_Pitch1.27mm, symbol 74AHC14
- removed R64: 301R, rklib:C0805-RES, symbol R
- removed R65: 100R, rklib:C0805-RES, symbol R
- removed R66, R67: 51R1, rklib:C0805-RES, symbol R
- removed R68: 1M00, rklib:C0805-RES, symbol R
- removed SW2: 5MS1, rklib:5MS1-SPDT, symbol Switch_SPDT
- removed X7: BNC, rklib:BNC-H, symbol BNC
- added B1, B2, B3, B4: TEST_1P, Mounting_Holes:MountingHole_3mm, symbol TEST_1P
- added C8, C9: 10u0./63V, Capacitors_ThroughHole:C_Radial_D5_L11_P2, symbol CP
- added IC1: LM1117-5.0, SOT-223, symbol LM1117-5.0
- added X7: MM-6G, rklib:MM-6G, symbol CONN_02X03
- SW1: footprint rklib:NT04-H -> Buttons_Switches_ThroughHole:SW_DIP_x4_Slide
Connections:
- net +12V: now also C8.1, IC1.3 (IN)
- net +3V3: now also X7.1 (P1)
- net +5V: now also C9.1, IC1.2 (OUT), IC1.4 (OUT), X7.2 (P2)
- net GND: now also C8.2, C9.2, IC1.1 (GND), X7.4 (P4), X7.6 (P6)
- net LRCK:1: now also R8.6 (R3); no longer R8.7 (R2)
- net MCLK:1: now also R8.7 (R2); no longer R8.8 (R1)
- net MDO:4: now also IC11.142 (IO_L2P_0); no longer IC11.143 (IO_L1N_VREF_0)
- net SCL:1: now also IC11.34 (IO_L1N_VREF_3); no longer IC11.35 (IO_L1P_3)
- net SCL:2: now also IC11.24 (IO_L41P_GCLK27_3); no longer IC11.26 (IO_L37N_3)
- net SCL:3: now also IC11.14 (IO_L44N_GCLK20_3); no longer IC11.15 (IO_L44P_GCLK21_3)
- net SCL:4: now also IC11.6 (IO_L52P_3); no longer IC11.7 (IO_L51N_3)
- net SDA:1: now also IC11.35 (IO_L1P_3); no longer IC11.34 (IO_L1N_VREF_3)
- net SDA:2: now also IC11.26 (IO_L37N_3); no longer IC11.24 (IO_L41P_GCLK27_3)
- net SDA:3: now also IC11.15 (IO_L44P_GCLK21_3); no longer IC11.14 (IO_L44N_GCLK20_3)
- net SDA:4: now also IC11.7 (IO_L51N_3); no longer IC11.6 (IO_L52P_3)
- net SW:1: now also R61.2, SW1.5; no longer R58.2, SW1.8
- net SW:2: now also R60.2, SW1.6; no longer R59.2, SW1.7
- net SW:3: now also R59.2, SW1.7; no longer R60.2, SW1.6
- net SW:4: now also R58.2, SW1.8; no longer R61.2, SW1.5
- net WCLKIN: now also IC11.102 (IO_L32P_1), X7.3 (P3); no longer IC11.114 (IO_L65N_SCP2_0)
- net WCLKOUT: now reaches IC11.101 (IO_L32N_1)
- net WCLKOUT: now also X7.5 (P5)
- net at R1.2: now also IC11.143 (IO_L1N_VREF_0); no longer IC11.142 (IO_L2P_0)
- net at IC11.32 (IO_L2N_3): now also R8.3 (P3); no longer R8.2 (P2)
- net at IC11.33 (IO_L2P_3): now also R8.2 (P2); no longer R8.1 (P1)
- no-connect marks 11 -> 15
Other:
- note removed: "Auf Tochterplatine auslagern"
- note removed: "TODO: 12V->5V"
- moved on the sheet: R1

Commit message: Reannotation
Parts:
- renumbered C84 to C1, C89 to C10, C90 to C11, C91 to C12, C92 to C13, C93 to C14, C94 to C15, C95 to C16, C96 to C17, C97 to C18, C98 to C19, C1 to C2, C99 to C20, C100 to C21, C101 to C22, C102 to C23, C103 to C24, C104 to C25, C105 to C26, C106 to C27, C107 to C28, C108 to C29, C2 to C3, C109 to C30, C8 to C31, C9 to C32, C85 to C33, C86 to C34, C87 to C35, C88 to C36, C3 to C4, C4 to C5, C83 to C6, C5 to C7, C6 to C8, C7 to C9, IC12 to IC1, IC11 to IC2, IC1 to IC3, IC20 to IC4, IC13 to IC5, JMP4 to JMP1, L3 to L1, L4 to L2, L5 to L3, L6 to L4, L1 to L5, L2 to L6, R48 to R1, R55 to R10, R9 to R11, R56 to R12, R10 to R13, R57 to R14, R58 to R15, R59 to R16, R60 to R17, R61 to R18, R49 to R19, R1 to R2, R80 to R20, R50 to R21, R51 to R22, R52 to R23, R53 to R24, R54 to R25, R2 to R3, R3 to R4, R4 to R5, R5 to R6, R6 to R7, R7 to R8, R8 to R9, X11 to X10, X12 to X11, X13 to X12, X6 to X13, X8 to X6, X9 to X7, X10 to X8, X7 to X9

Commit message: Changed Termination
Parts:
- added R26, R27, R28, R29, R30, R31, R32, R33, R34, R35, R36, R37, R39, R40, R41, R43, R44, R45: 33R0, Capacitors_SMD:C_0402, symbol R
- added R38, R42: 33R0, Resistors_SMD:R_Array_Convex_4x0603, symbol R_PACK4
- R11, R13, R2, R4, R6, R8: footprint rklib:C0805-RES -> Capacitors_SMD:C_0402
Connections:
- net BCLK:5: now also R38.3 (P3); no longer IC2.45 (IO_L49N_D4_2)
- net BCLK:6: now also R42.2 (P2); no longer IC2.57 (IO_L14N_D12_2)
- net LRCK:5: now also R38.4 (P4); no longer IC2.46 (IO_L49P_D3_2)
- net LRCK:6: now also R42.3 (P3); no longer IC2.58 (IO_L14P_D11_2)
- net MCLK:4: now also R3.7 (R2); no longer R3.8 (R1)
- net MCLK:5: now also R39.2; no longer IC2.50 (IO_L31N_GCLK30_D15_2)
- net MCLK:6: now also R45.2; no longer IC2.62 (IO_L12P_D1_MISO2_2)
- net MDO:1: now also R28.2; no longer IC2.29 (IO_L36N_3)
- net MDO:2: now also R31.2; no longer IC2.17 (IO_L43P_GCLK23_3)
- net MDO:3: now also R36.2; no longer IC2.9 (IO_L50N_3)
- net MDO:4: now also R37.1; no longer IC2.142 (IO_L2P_0)
- net MDO:5: now also R38.2 (P2); no longer IC2.44 (IO_L62P_D5_2)
- net MDO:6: now also R42.1 (P1); no longer IC2.56 (IO_L30P_GCLK1_D13_2)
- net SCL:1: now also R32.2; no longer IC2.34 (IO_L1N_VREF_3)
- net SCL:2: now also R26.2; no longer IC2.24 (IO_L41P_GCLK27_3)
- net SCL:3: now also R29.2; no longer IC2.14 (IO_L44N_GCLK20_3)
- net SCL:4: now also R34.2; no longer IC2.6 (IO_L52P_3)
- net SCL:5: now also R41.2; no longer IC2.48 (IO_L48P_D7_2)
- net SCL:6: now also R44.2; no longer IC2.61 (IO_L12N_D2_MISO3_2)
- net SDA:1: now also R33.2; no longer IC2.35 (IO_L1P_3)
- net SDA:2: now also R27.2; no longer IC2.26 (IO_L37N_3)
- net SDA:3: now also R30.2; no longer IC2.15 (IO_L44P_GCLK21_3)
- net SDA:4: now also R35.2; no longer IC2.7 (IO_L51N_3)
- net SDA:5: now also R40.2; no longer IC2.47 (IO_L48N_RDWR_B_VREF_2)
- net SDA:6: now also R43.2; no longer IC2.59 (IO_L13N_D10_2)
- net at IC2.41 (IO_L64P_D8_2): now also R13.1
- net at IC2.43 (IO_L62N_D6_2): now also R38.7 (R2); no longer R13.1
- net at IC2.5 (IO_L52N_3): now also R3.2 (P2); no longer R3.1 (P1)
- new net: IC2.14 (IO_L44N_GCLK20_3), R29.1
- new net: IC2.142 (IO_L2P_0), R37.2
- new net: IC2.15 (IO_L44P_GCLK21_3), R30.1
- new net: IC2.17 (IO_L43P_GCLK23_3), R31.1
- new net: IC2.24 (IO_L41P_GCLK27_3), R26.1
- new net: IC2.26 (IO_L37N_3), R27.1
- new net: IC2.29 (IO_L36N_3), R28.1
- new net: IC2.34 (IO_L1N_VREF_3), R32.1
- new net: IC2.35 (IO_L1P_3), R33.1
- new net: IC2.44 (IO_L62P_D5_2), R38.6 (R3)
- new net: IC2.45 (IO_L49N_D4_2), R38.5 (R4)
- new net: IC2.47 (IO_L48N_RDWR_B_VREF_2), R40.1
- new net: IC2.48 (IO_L48P_D7_2), R41.1
- new net: IC2.50 (IO_L31N_GCLK30_D15_2), R39.1
- new net: IC2.56 (IO_L30P_GCLK1_D13_2), R42.8 (R1)
- new net: IC2.57 (IO_L14N_D12_2), R42.7 (R2)
- new net: IC2.58 (IO_L14P_D11_2), R42.6 (R3)
- new net: IC2.59 (IO_L13N_D10_2), R43.1
- new net: IC2.6 (IO_L52P_3), R34.1
- new net: IC2.61 (IO_L12N_D2_MISO3_2), R44.1
- new net: IC2.62 (IO_L12P_D1_MISO2_2), R45.1
- new net: IC2.7 (IO_L51N_3), R35.1
- new net: IC2.9 (IO_L50N_3), R36.1
- no-connect marks 15 -> 17
