File: SOURCES/KICAD/ADAT-IO-x4.kicad_pcb (KiCad board)
At the start: 2 copper layers, 100 x 100 mm, 123 parts, among them J1 Barrel_Jack_Switch, J10 Conn_02x11_Odd_Even, J11 Conn_02x10_Odd_Even, J12 Conn_02x08_Odd_Even, J13 Conn_02x08_Odd_Even, J14 Conn_02x08_Odd_Even, J15 Conn_02x08_Odd_Even, J2 Barrel_Jack_Switch, J3 Conn_02x08_Odd_Even, J4 Conn_02x08_Odd_Even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

Commit message: ADATA-IO-x4 ki-CAD Initial Release version 0.2
Parts:
- added J16: Conn_01x02, Connector_PinHeader_2.54mm:PinHeader_1x02_P2.54mm_Vertical, F.Cu at (148.8, 94.4)
- R11, R15, R17, R9: value NOP -> 100k
- R36: value 100k -> 3.3k
- R60: value 100K -> 10k
- moved R8 0.97 mm to (227.4, 121.8)
- moved R60 0.77 mm to (211.2, 93.2)
Connections:
- J3 pad 7: BCLKin -> Net-(J3-Pad7)
- J4 pad 7: BCLKin -> Net-(J4-Pad7)
- J6 pad 7: BCLKin -> Net-(J6-Pad7)
- R11 pad 1: Net-(J4-Pad9) -> DATAin3
- R11 pad 2: LRCLKin -> GND
- R15 pad 1: Net-(J6-Pad9) -> DATAin1
- R15 pad 2: LRCLKin -> GND
- R9 pad 1: Net-(J3-Pad9) -> DATAin2
- R9 pad 2: LRCLKin -> GND
- U8 pad 2: GNDD -> +5VD
Routing:
- net Net-(J3-Pad9): track 19.8 -> 0.00 mm
- net Net-(J4-Pad9): track 19.8 -> 0.00 mm
- net Net-(J6-Pad9): track 18.8 -> 0.00 mm
- net DATAin2: track 63.7 -> 78.6 mm
- net DATAin3: track 49.9 -> 64.8 mm
- net DATAin1: track 58.3 -> 72.0 mm
- net /ADATx4RX-Part/SMUX: track 6.53 -> 15.0 mm
- net BCLKin: track 83.3 -> 81.0 mm
- net GNDD: track 58.8 -> 57.4 mm, vias 24 -> 23
- net ~RX_RES: track 43.6 -> 44.9 mm
- net LRCLKin: track 104.5 -> 103.4 mm
- net +3V3: track 63.0 -> 64.0 mm
- net /ADATx4TX-Part/~TX_MUTE: track 20.8 -> 21.6 mm
- net VIN: track 87.6 -> 88.4 mm
- net DAC_SCL: track 72.8 -> 73.4 mm
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Other:
- board text added: "Designed by CyberPit 2021"
- board text added: "OUT0"
- board text added: "OUT1"
- board text added: "OUT2"
- board text added: "SMUX-IN"
- board text added: "SMUX-OUT"
- board text added: "~MUTE"
