File: SOURCES/KICAD/ADATx4RX-Part.sch (KiCad schematic (older format))
At the start: 59 parts, among them J10 Conn_02x11_Odd_Even, J11 Conn_02x10_Odd_Even, J12 Conn_02x08_Odd_Even, J13 Conn_02x08_Odd_Even, J14 Conn_02x08_Odd_Even, J15 Conn_02x08_Odd_Even, Q2 2N7002, U10 74LVC541A, U6 PLT133/T10W, U7 PLR135/T10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

Commit message: ADATA-IO-x4 ki-CAD Initial Release version 0.2
Parts:
- added J16: Conn_01x02, Connector_PinHeader_2.54mm:PinHeader_1x02_P2.54mm_Vertical, symbol Connector_Generic:Conn_01x02
Connections:
- net +5VD: now also U8.2
- net GNDD: now also J16.1 (Pin_1); no longer U8.2
- net SMUX: now also J16.2 (Pin_2)
Other:
- note added: "*Inverted (since ver0.2)"
- note added: "SMUX"
- note added: "SMUX-OUT"
- note added: "This is general pourpse output\n(ex. Manual Reset/Mute/One-way-UART communication, etc…)"
- note removed: "MUTE"
Changed lines of the file:
@@
 Sheet 3 3
 Title "ADAT I8S Reciever Part"
-Date "2021-02-11"
-Rev "0.1"
+Date "2021-08-01"
+Rev "0.2"
 Comp "CyberPit HILO. 2021"
 Comment1 ""
@@
 	1    0    0    -1
 $EndComp
-Text Label 1075 1175 0    50   ~ 0
+Text Label 825  1175 0    50   ~ 0
 BCLK
 Wire Wire Line
@@
 U 1 1 60F7D790
 P 6950 5100
-F 0 "R47" V 6900 5300 50  0000 C CNN
+F 0 "R47" V 6800 5100 50  0000 C CNN
 F 1 "33" V 6950 5100 50  0000 C CNN
 F 2 "fdsp_resistor:R_0805_HandSoldering" V 6880 5100 50  0001 C CNN
@@
 U 1 1 60F8DDED
 P 6950 5200
-F 0 "R48" V 7000 5400 50  0000 C CNN
+F 0 "R48" V 7100 5200 50  0000 C CNN
 F 1 "33" V 6950 5200 50  0000 C CNN
 F 2 "fdsp_resistor:R_0805_HandSoldering" V 6880 5200 50  0001 C CNN
@@
 U 1 1 6140B425
 P 4550 4850
-F 0 "R28" V 4500 5000 50  0000 C CNN
+F 0 "R28" V 4450 4850 50  0000 C CNN
 F 1 "33" V 4550 4850 50  0000 C CNN
 F 2 "fdsp_resistor:R_0805_HandSoldering" V 4480 4850 50  0001 C CNN
@@
 AR Path="/60262604/6174C38E" Ref="R?"  Part="1"
 AR Path="/60262E22/6174C38E" Ref="R46"  Part="1"
-F 0 "R46" V 5050 4750 50  0000 C CNN
+F 0 "R46" V 5025 4950 50  0000 C CNN
 F 1 "3.3k" V 5100 4950 50  0000 C CNN
 F 2 "fdsp_resistor:R_0805_HandSoldering" V 5030 4950 50  0001 C CNN
@@
 	5000 4480 4600 4480
 Text Notes 4230 7210 0    79   ~ 16
-MUTE
+SMUX
 Wire Notes Line style solid
 	4200 7050 4200 7250
@@
 $EndComp
 Connection ~ 4950 5600
-Text Label 1050 1650 0    50   ~ 0
+Text Label 800  1650 0    50   ~ 0
 LRCK
 Wire Wire Line
@@
 	9600 5375 9850 5375
 Wire Wire Line
-	1075 1175 1325 1175
+	825  1175 1325 1175
 Text Label 2450 1075 2    50   ~ 0
 ~BCLK
@@
 	1250 3500 1250 3400
 Wire Wire Line
-	1250 1850 1350 1850
-Wire Wire Line
 	1350 2550 1250 2550
-Connection ~ 1250 2550
 Wire Wire Line
 	1350 3200 1250 3200
@@
 	1175 975  1325 975
 Wire Wire Line
-	1350 1650 1050 1650
+	1350 1650 800  1650
 Wire Wire Line
 	1950 1750 2450 1750
@@
 Wire Wire Line
 	1250 3200 1250 3400
-Wire Wire Line
-	1250 1850 1250 2550
 Wire Wire Line
 	875  2350 1350 2350
@@
 Wire Wire Line
 	4850 2400 4650 2400
+Wire Wire Line
+	1175 975  1175 1850
+Wire Wire Line
+	1175 1850 1350 1850
+Connection ~ 1175 975
+Text Notes 1900 1900 0    50   ~ 0
+*Inverted (since ver0.2)
+$Comp
+L Connector_Generic:Conn_01x02 J16
+U 1 1 61451684
+P 5450 6700
+F 0 "J16" H 5400 6350 50  0000 C CNN
+F 1 "Conn_01x02" H 5400 6450 50  0000 C CNN
+F 2 "Connector_PinHeader_2.54mm:PinHeader_1x02_P2.54mm_Vertical" H 5450 6700 50  0001 C CNN
+F 3 "~" H 5450 6700 50  0001 C CNN
+	1    5450 6700
+	1    0    0    1
+$EndComp
+$Comp
+L fdsp_power:GNDD #PWR071
+U 1 1 61454577
+P 5150 6775
+F 0 "#PWR071" H 5150 6525 50  0001 C CNN
+F 1 "GNDD" H 5150 6625 50  0000 C CNN
+F 2 "" H 5150 6775 60  0000 C CNN
+F 3 "" H 5150 6775 60  0000 C CNN
+	1    5150 6775
+	1    0    0    -1
+$EndComp
+Wire Wire Line
+	5150 6775 5150 6700
+Wire Wire Line
+	5150 6700 5250 6700
+Text Notes 5630 6710 0    79   ~ 16
+SMUX-OUT
+Wire Notes Line style solid
+	5625 6550 5625 6725
+Wire Notes Line style solid
+	5625 6725 6325 6725
+Wire Notes Line style solid
+	6325 6725 6325 6550
+Wire Notes Line style solid
+	6325 6550 5625 6550
+Text Notes 5700 6450 0    50   ~ 0
+This is general pourpse output\n(ex. Manual Reset/Mute/One-way-UART communication, etc…)
 $EndSCHEMATC
