File: SOURCES/KICAD/ADATx4TX-Part.sch (KiCad schematic (older format))
At the start: 42 parts, among them J3 Conn_02x08_Odd_Even, J4 Conn_02x08_Odd_Even, J5 Conn_02x08_Odd_Even, J6 Conn_02x08_Odd_Even, J7 Conn_02x11_Odd_Even, J8 Conn_02x10_Odd_Even, J9 Conn_01x02, Q1 AO3401A, U3 74HCT541, U4 V1401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

Commit message: R36 value changed to 3k3
Parts:
- R36: value 100k -> 3.3k
Changed lines of the file:
@@
 P 8725 4800
 F 0 "R36" V 8625 4800 50  0000 C CNN
-F 1 "100k" V 8725 4800 50  0000 C CNN
+F 1 "3.3k" V 8725 4800 50  0000 C CNN
 F 2 "fdsp_resistor:R_0805_HandSoldering" V 8655 4800 50  0001 C CNN
 F 3 "~" H 8725 4800 50  0001 C CNN

Commit message: ADATA-IO-x4 ki-CAD Initial Release version 0.2
Parts:
- R11, R15, R17, R9: value NOP -> 100k
- R24: value 100k -> 10k
- R60: value 100K -> 10k
Connections:
- net BCLKin: no longer J3.7 (Pin_7), J4.7 (Pin_7), J6.7 (Pin_7)
- net DATAin1: now also R15.1
- net DATAin2: now also R9.1
- net DATAin3: now also R11.1
- net GND: now also R11.2, R15.2, R9.2
- net LRCLKin: no longer R11.2, R15.2, R9.2
- net at J6.9 (Pin_9): no longer R15.1
- net at J3.9 (Pin_9): no longer R9.1
- net at J4.9 (Pin_9): no longer R11.1
Other:
- note added: "*Pull down I8S Data-Lines for stability (since 0v2)"
- note added: "*Valuse Changed for Stability"
- note added: "H: MUTE\nL: 24bit(23bit I2S) Left Justified"
- note removed: "H: MUTE\nL: 24bit Left Justified"
- moved on the sheet: R11, R15, R9
Changed lines of the file:
@@
 Sheet 2 3
 Title "ADAT Format I8S Optical Transmitter Part"
-Date "2021-02-11"
-Rev "0.1"
+Date "2021-08-01"
+Rev "0.2"
 Comp "Designed  by CyberPit HILO. 2020"
 Comment1 ""
@@
 U 1 1 6038F86A
 P 4850 6050
-F 0 "J8" H 4550 7000 50  0000 C CNN
-F 1 "Conn_02x10_Odd_Even" H 4925 6925 50  0000 C CNN
+F 0 "J8" H 4550 7025 50  0000 C CNN
+F 1 "Conn_02x10_Odd_Even" H 4925 6950 50  0000 C CNN
 F 2 "Connector_IDC:IDC-Header_2x10_P2.54mm_Vertical" H 4850 6050 50  0001 C CNN
 F 3 "~" H 4850 6050 50  0001 C CNN
@@
 Text GLabel 2200 5150 0    51   Output ~ 0
 MCLKin
-Text GLabel 2200 4850 0    51   Output ~ 0
-LRCLKin
 $Comp
 L Device:R R9
 U 1 1 6074CC36
-P 2500 4850
-F 0 "R9" V 2450 4650 50  0000 C CNN
-F 1 "NOP" V 2500 4850 50  0000 C CNN
-F 2 "fdsp_resistor:R_0805_HandSoldering" V 2430 4850 50  0001 C CNN
-F 3 "~" H 2500 4850 50  0001 C CNN
-	1    2500 4850
+P 2150 4250
+F 0 "R9" V 2050 4250 50  0000 C CNN
+F 1 "100k" V 2150 4250 50  0000 C CNN
+F 2 "fdsp_resistor:R_0805_HandSoldering" V 2080 4250 50  0001 C CNN
+F 3 "~" H 2150 4250 50  0001 C CNN
+	1    2150 4250
 	0    1    1    0
 $EndComp
@@
 $EndComp
 Wire Wire Line
-	2200 4850 2350 4850
-Wire Wire Line
 	2350 5150 2200 5150
 Text GLabel 2200 6650 0    51   Output ~ 0
 MCLKin
-Text GLabel 2200 6350 0    51   Output ~ 0
-LRCLKin
 $Comp
 L Device:R R11
 U 1 1 6075000A
-P 2500 6350
-F 0 "R11" V 2450 6150 50  0000 C CNN
-F 1 "NOP" V 2500 6350 50  0000 C CNN
-F 2 "fdsp_resistor:R_0805_HandSoldering" V 2430 6350 50  0001 C CNN
-F 3 "~" H 2500 6350 50  0001 C CNN
-	1    2500 6350
+P 2125 5750
+F 0 "R11" V 2000 5725 50  0000 C CNN
+F 1 "100k" V 2125 5750 50  0000 C CNN
+F 2 "fdsp_resistor:R_0805_HandSoldering" V 2055 5750 50  0001 C CNN
+F 3 "~" H 2125 5750 50  0001 C CNN
+	1    2125 5750
 	0    1    1    0
 $EndComp
@@
 $EndComp
 Wire Wire Line
-	2200 6350 2350 6350
-Wire Wire Line
 	2350 6650 2200 6650
 Text GLabel 2250 3800 0    51   Output ~ 0
 MCLKin
-Text GLabel 2250 3500 0    51   Output ~ 0
-LRCLKin
 $Comp
 L Device:R R15
 U 1 1 607542A0
-P 2550 3500
-F 0 "R15" V 2500 3300 50  0000 C CNN
-F 1 "NOP" V 2550 3500 50  0000 C CNN
-F 2 "fdsp_resistor:R_0805_HandSoldering" V 2480 3500 50  0001 C CNN
-F 3 "~" H 2550 3500 50  0001 C CNN
-	1    2550 3500
+P 2275 2950
+F 0 "R15" V 2175 2950 50  0000 C CNN
+F 1 "100k" V 2275 2950 50  0000 C CNN
+F 2 "fdsp_resistor:R_0805_HandSoldering" V 2205 2950 50  0001 C CNN
+F 3 "~" H 2275 2950 50  0001 C CNN
+	1    2275 2950
 	0    1    1    0
 $EndComp
@@
 $EndComp
 Wire Wire Line
-	2250 3500 2400 3500
-Wire Wire Line
 	2400 3800 2250 3800
 $Comp
@@
 Text GLabel 2700 1800 0    51   Input ~ 0
 ADCDout0
-Text GLabel 2650 4550 0    51   Input ~ 0
+Text GLabel 2300 4550 0    51   Input ~ 0
 ADCDout2
-Text GLabel 2650 6050 0    51   Input ~ 0
+Text GLabel 2275 6050 0    51   Input ~ 0
 ADCDout3
-Text GLabel 2700 3200 0    51   Input ~ 0
+Text GLabel 2325 3200 0    51   Input ~ 0
 ADCDout1
-Text GLabel 2250 3400 0    51   Output ~ 0
-BCLKin
-Wire Wire Line
-	2250 3400 2700 3400
 Text GLabel 2250 2000 0    51   Output ~ 0
 BCLKin
 Wire Wire Line
 	2250 2000 2700 2000
-Text GLabel 2200 4750 0    51   Output ~ 0
-BCLKin
-Wire Wire Line
-	2200 4750 2650 4750
-Text GLabel 2200 6250 0    51   Output ~ 0
-BCLKin
-Wire Wire Line
-	2200 6250 2650 6250
 Text GLabel 2200 5050 0    51   BiDi ~ 0
 SCL
@@
 	2250 3700 2700 3700
 Wire Wire Line
-	2250 3300 2700 3300
-Wire Wire Line
-	2200 6150 2650 6150
-Wire Wire Line
-	2200 4650 2650 4650
+	2250 3300 2475 3300
+Wire Wire Line
+	2200 6150 2400 6150
+Wire Wire Line
+	2200 4650 2400 4650
 Wire Wire Line
 	2250 1900 2700 1900
@@
 P 8650 3450
 F 0 "R24" V 8550 3450 50  0000 C CNN
-F 1 "100k" V 8650 3450 50  0000 C CNN
+F 1 "10k" V 8650 3450 50  0000 C CNN
 F 2 "fdsp_resistor:R_0805_HandSoldering" V 8580 3450 50  0001 C CNN
 F 3 "~" H 8650 3450 50  0001 C CNN
@@
 $EndComp
 Text Notes 8700 3150 0    50   ~ 0
-H: MUTE\nL: 24bit Left Justified
+H: MUTE\nL: 24bit(23bit I2S) Left Justified
 $Comp
 L Transistor_FET:AO3401A Q1
@@
 Text Notes 2600 6750 0    75   ~ 0
 #
-Text Notes 2600 6450 0    75   ~ 0
-#
 Wire Wire Line
 	5200 6150 5200 6700
@@
 P 5450 1700
 F 0 "R17" V 5350 1700 50  0000 C CNN
-F 1 "NOP" V 5450 1700 50  0000 C CNN
+F 1 "100k" V 5450 1700 50  0000 C CNN
 F 2 "fdsp_resistor:R_0805_HandSoldering" V 5380 1700 50  0001 C CNN
 F 3 "~" H 5450 1700 50  0001 C CNN
@@
 P 4675 5425
 F 0 "R60" V 4575 5425 50  0000 C CNN
-F 1 "100K" V 4675 5425 50  0000 C CNN
+F 1 "10k" V 4675 5425 50  0000 C CNN
 F 2 "fdsp_resistor:R_0805_HandSoldering" V 4605 5425 50  0001 C CNN
 F 3 "~" H 4675 5425 50  0001 C CNN
@@
 Text Label 3650 5950 0    50   ~ 0
 ~TX_MUTE
+Wire Wire Line
+	2425 2950 2475 2950
+$Comp
+L power:GND #PWR070
+U 1 1 6160AA9E
+P 2025 2950
+F 0 "#PWR070" H 2025 2700 50  0001 C CNN
+F 1 "GND" H 2025 2800 50  0000 C CNN
+F 2 "" H 2025 2950 50  0000 C CNN
+F 3 "" H 2025 2950 50  0000 C CNN
+	1    2025 2950
+	1    0    0    -1
+$EndComp
+Wire Wire Line
+	2025 2950 2125 2950
+Wire Wire Line
+	2300 4250 2400 4250
+$Comp
+L power:GND #PWR069
+U 1 1 61684F6A
+P 1900 4250
+F 0 "#PWR069" H 1900 4000 50  0001 C CNN
+F 1 "GND" H 1900 4100 50  0000 C CNN
+F 2 "" H 1900 4250 50  0000 C CNN
+F 3 "" H 1900 4250 50  0000 C CNN
+	1    1900 4250
+	1    0    0    -1
+$EndComp
+Wire Wire Line
+	1900 4250 2000 4250
+Wire Wire Line
+	2325 3200 2700 3200
+Wire Wire Line
+	2300 4550 2650 4550
+Wire Wire Line
+	2475 2950 2475 3300
+Connection ~ 2475 3300
+Wire Wire Line
+	2475 3300 2700 3300
+Wire Wire Line
+	2400 4250 2400 4650
+Connection ~ 2400 4650
+Wire Wire Line
+	2400 4650 2650 4650
+Wire Wire Line
+	2275 5750 2400 5750
+$Comp
+L power:GND #PWR021
+U 1 1 6174A40B
+P 1875 5750
+F 0 "#PWR021" H 1875 5500 50  0001 C CNN
+F 1 "GND" H 1875 5600 50  0000 C CNN
+F 2 "" H 1875 5750 50  0000 C CNN
+F 3 "" H 1875 5750 50  0000 C CNN
+	1    1875 5750
+	1    0    0    -1
+$EndComp
+Wire Wire Line
+	1875 5750 1975 5750
+Wire Wire Line
+	2275 6050 2650 6050
+Wire Wire Line
+	2400 5750 2400 6150
+Connection ~ 2400 6150
+Wire Wire Line
+	2400 6150 2650 6150
+Text Notes 1975 975  0    50   ~ 0
+*Pull down I8S Data-Lines for stability (since 0v2)
+Text Notes 3450 5300 0    50   ~ 0
+*Valuse Changed for Stability
+Text Notes 4525 5425 0    50   ~ 0
+*
+Text Notes 8800 3500 0    50   ~ 0
+*Valuse Changed for Stability
 $EndSCHEMATC
